File: Pong.kicad_pcb (KiCad board)
At the start: 2 copper layers, 107.9 x 61.5 mm, 43 parts, among them J1 RCJ-013, J2 RCJ-013, J3 Barrel_Jack, J4 Atari Paddle Port 1, J5 Atari Paddle Port 2, SW1 SW_Rotary_1x7_MP, SW2 Reset, SW3 angle, SW4 speed, SW5 serve, SW6 bat_size, SW7 SW_SPDT, U1 7805, U2 L7806, U3 AY-3-8500, X1 2MHz

Commit message: Gerbers
Parts:
- renumbered G*** to G1
Other:
- board text added: "{dblquote}Pong Video Game{dblquote} https://github.com/madcatse/Pong-by-MadCat Made by MadCat, 2025 Version 1.0 https://t.me/madcatse www.youtube.com/@MadCatSE"
- board text removed: "{dblquote}Pong Video Game{dblquote} Made by MadCat, 2025 Version 1.0 https://t.me/madcatse www.youtube.com/@MadCatSE"
Changed lines of the file:
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@@
     (at 157.226 73.9902)
     (attr board_only exclude_from_pos_files exclude_from_bom allow_missing_courtyard)
-    (fp_text reference "G***" (at 0.06 5.72) (layer "F.SilkS") hide
+    (fp_text reference "G1" (at 0.06 5.72) (layer "F.SilkS") hide
         (effects (font (size 1.5 1.5) (thickness 0.3)))
     )
@@
     (tags "mounting hole 2.7mm no annular m2.5")
     (attr board_only exclude_from_pos_files exclude_from_bom)
-    (fp_text reference "H2" (at -0.0254 2.6162) (layer "F.SilkS")
+    (fp_text reference "H2" (at -0.0508 -2.3876) (layer "F.SilkS")
         (effects (font (size 1 1) (thickness 0.15)))
     )
@@
     (property "ki_keywords" "switch lever")
     (attr through_hole)
-    (fp_text reference "SW3" (at 0.1524 5.4356 90) (layer "F.SilkS")
+    (fp_text reference "SW3" (at -0.0508 -2.2098 90) (layer "F.SilkS")
         (effects (font (size 1 1) (thickness 0.15)))
     )
@@
         (effects (font (size 1 1) (thickness 0.15)))
     )
-    (fp_text value "1N4148" (at 5.334 -1.6764) (layer "F.SilkS")
+    (fp_text value "1N4148" (at 5.08 1.7018) (layer "F.SilkS")
         (effects (font (size 0.75 0.75) (thickness 0.1)))
     )
-    (fp_text user "K" (at 0 -1.8) (layer "F.SilkS")
+    (fp_text user "K" (at 1.4986 -0.8128) (layer "F.SilkS")
         (effects (font (size 1 1) (thickness 0.15)))
     )
@@
     (property "ki_keywords" "switch lever")
     (attr through_hole)
-    (fp_text reference "SW5" (at 0.1524 5.4356 90) (layer "F.SilkS")
+    (fp_text reference "SW5" (at 0 -2.2098 90) (layer "F.SilkS")
         (effects (font (size 1 1) (thickness 0.15)))
     )
@@
     (tags "mounting hole 2.7mm no annular m2.5")
     (attr board_only exclude_from_pos_files exclude_from_bom)
-    (fp_text reference "H1" (at -4.191 -0.1016) (layer "F.SilkS")
+    (fp_text reference "H1" (at -0.0508 -2.5654) (layer "F.SilkS")
         (effects (font (size 1 1) (thickness 0.15)))
     )
@@
     (property "ki_keywords" "switch lever")
     (attr through_hole)
-    (fp_text reference "SW4" (at 0.1524 5.4356 90) (layer "F.SilkS")
+    (fp_text reference "SW4" (at 0.0508 -2.159 90) (layer "F.SilkS")
         (effects (font (size 1 1) (thickness 0.15)))
     )
@@
     (tags "mounting hole 2.7mm no annular m2.5")
     (attr board_only exclude_from_pos_files exclude_from_bom)
-    (fp_text reference "H4" (at -3.7846 -0.0254 -90) (layer "F.SilkS")
+    (fp_text reference "H4" (at -0.0508 -2.3876) (layer "F.SilkS")
         (effects (font (size 1 1) (thickness 0.15)))
     )
@@
     (property "ki_keywords" "switch normally-open pushbutton push-button")
     (attr through_hole)
-    (fp_text reference "SW2" (at 0.1524 5.4356 90) (layer "F.SilkS")
+    (fp_text reference "SW2" (at 0.0508 -2.2352 90) (layer "F.SilkS")
         (effects (font (size 1 1) (thickness 0.15)))
     )
@@
     (property "ki_keywords" "switch lever")
     (attr through_hole)
-    (fp_text reference "SW6" (at 0.1524 5.4356 90) (layer "F.SilkS")
+    (fp_text reference "SW6" (at 0.0254 -2.2606 90) (layer "F.SilkS")
         (effects (font (size 1 1) (thickness 0.15)))
     )
-    (fp_text value "bat_size" (at 3.0226 1.524 180) (layer "F.SilkS")
+    (fp_text value "bat_size" (at 2.4892 1.3716 180) (layer "F.SilkS")
         (effects (font (size 1 1) (thickness 0.15)))
     )
@@
     (tags "mounting hole 2.7mm no annular m2.5")
     (attr board_only exclude_from_pos_files exclude_from_bom)
-    (fp_text reference "H3" (at 0 -3.7) (layer "F.SilkS")
+    (fp_text reference "H3" (at 0.0508 -2.5654) (layer "F.SilkS")
         (effects (font (size 1 1) (thickness 0.15)))
     )
@@
   (gr_rect (start 84.0232 31.6992) (end 191.9478 93.1926)
     (stroke (width 0.05) (type default)) (fill none) (layer "Edge.Cuts"))
-  (gr_text "{dblquote}Pong Video Game{dblquote}\nMade by MadCat, 2025\nVersion 1.0\nhttps://t.me/madcatse\nwww.youtube.com/@MadCatSE" (at 123.3678 66.5988) (layer "B.SilkS")
+  (gr_text "{dblquote}Pong Video Game{dblquote}\nhttps://github.com/madcatse/Pong-by-MadCat\nMade by MadCat, 2025\nVersion 1.0\nhttps://t.me/madcatse\nwww.youtube.com/@MadCatSE" (at 132.3848 68.7324) (layer "B.SilkS")
     (effects (font (size 1 1) (thickness 0.15)) (justify left bottom mirror))
   )
@@
   (segment (start 117.5297 53.6323) (end 118.0846 54.1872) (width 0.2) (layer "B.Cu") (net 16))
   (segment (start 118.0846 70.0435) (end 119.3546 71.3135) (width 0.2) (layer "B.Cu") (net 16))
-  (segment (start 126.2966 87.9697) (end 125.1387 86.8118) (width 0.2) (layer "F.Cu") (net 17))
   (segment (start 102.9346 87.9697) (end 98.2053 83.2404) (width 0.2) (layer "F.Cu") (net 17))
-  (segment (start 126.2966 87.9697) (end 126.2966 88.1966) (width 0.2) (layer "F.Cu") (net 17))
-  (segment (start 114.665 86.8118) (end 113.5071 87.9697) (width 0.2) (layer "F.Cu") (net 17))
-  (segment (start 148.2557 87.9697) (end 126.2966 87.9697) (width 0.2) (layer "F.Cu") (net 17))
+  (segment (start 126.365 88.265) (end 126.2966 88.1966) (width 0.2) (layer "F.Cu") (net 17))
+  (segment (start 148.2557 87.9697) (end 126.9905 87.9697) (width 0.2) (layer "F.Cu") (net 17))
   (segment (start 113.5071 87.9697) (end 102.9346 87.9697) (width 0.2) (layer "F.Cu") (net 17))
-  (segment (start 125.1387 86.8118) (end 114.665 86.8118) (width 0.2) (layer "F.Cu") (net 17))
+  (segment (start 114.665 86.8118) (end 113.5071 87.9697) (width 0.2) (layer "F.Cu") (net 17))
+  (segment (start 126.6952 88.265) (end 126.365 88.265) (width 0.2) (layer "F.Cu") (net 17))
   (segment (start 97.0534 83.2404) (end 98.2053 83.2404) (width 0.2) (layer "F.Cu") (net 17))
+  (segment (start 126.9905 87.9697) (end 126.6952 88.265) (width 0.2) (layer "F.Cu") (net 17))
+  (segment (start 126.2966 88.1966) (end 124.9118 86.8118) (width 0.2) (layer "F.Cu") (net 17))
+  (segment (start 124.9118 86.8118) (end 114.665 86.8118) (width 0.2) (layer "F.Cu") (net 17))
   (via (at 126.2966 88.1966) (size 0.6) (drill 0.3) (layers "F.Cu" "B.Cu") (net 17))
   (segment (start 126.2966 80.942) (end 131.5466 75.692) (width 0.2) (layer "B.Cu") (net 17))
@@
   (segment (start 104.3346 71.0596) (end 105.5527 72.2777) (width 0.2) (layer "F.Cu") (net 21))
   (segment (start 88.8327 64.4398) (end 88.8327 64.7279) (width 0.2) (layer "F.Cu") (net 22))
-  (segment (start 114.8921 85.1297) (end 117.6621 85.1297) (width 0.2) (layer "F.Cu") (net 22))
   (segment (start 113.1727 72.1871) (end 113.1727 72.4154) (width 0.2) (layer "F.Cu") (net 22))
   (segment (start 117.6621 85.1297) (end 120.1148 82.677) (width 0.2) (layer "F.Cu") (net 22))
@@
   (segment (start 147.188 82.677) (end 149.6407 85.1297) (width 0.2) (layer "F.Cu") (net 22))
   (segment (start 120.1148 82.677) (end 147.188 82.677) (width 0.2) (layer "F.Cu") (net 22))
-  (segment (start 152.4107 85.1297) (end 149.6407 85.1297) (width 0.2) (layer "F.Cu") (net 22))
   (segment (start 89.6965 65.5917) (end 106.5773 65.5917) (width 0.2) (layer "F.Cu") (net 22))
   (segment (start 114.2746 72.4154) (end 113.1727 72.4154) (width 0.2) (layer "F.Cu") (net 22))
+  (segment (start 114.8921 85.1297) (end 117.6621 85.1297) (width 0.2) (layer "B.Cu") (net 22))
   (segment (start 114.2746 84.5122) (end 114.8921 85.1297) (width 0.2) (layer "B.Cu") (net 22))
   (segment (start 114.2746 72.4154) (end 114.2746 84.5122) (width 0.2) (layer "B.Cu") (net 22))
+  (segment (start 149.6407 85.1297) (end 152.4107 85.1297) (width 0.2) (layer "B.Cu") (net 22))
   (segment (start 123.3327 72.4154) (end 123.3327 72.5533) (width 0.2) (layer "F.Cu") (net 23))
   (segment (start 124.4346 72.4154) (end 123.3327 72.4154) (width 0.2) (layer "F.Cu") (net 23))
